File: Milpitas/powerInput.sch (KiCad schematic (older format))
At the start: 61 parts

Commit message: Updated some silly mistakes
Updated some silly mistakes,
- capacitor decoupled to gnd
- Added option for jumper control to 2 24V modules
Parts:
- removed R?: 1k, symbol Device:R
- C? (x12): symbol Device:C_Small -> Milpitas-rescue:C_Small-Device
- D?: symbol Device:D_TVS -> Milpitas-rescue:D_TVS-Device
- D?: symbol Device:D_Zener -> Milpitas-rescue:D_Zener-Device
- D?: symbol Device:Q_SCR_AGK -> Milpitas-rescue:Q_SCR_AGK-Device
- D? (x2): symbol Device:LED -> Milpitas-rescue:LED-Device
- F?: symbol Device:Fuse -> Milpitas-rescue:Fuse-Device
- FB?: symbol Device:Ferrite_Bead -> Milpitas-rescue:Ferrite_Bead-Device
- J?: symbol Connector:Conn_01x02_Female -> Milpitas-rescue:Conn_01x02_Female-Connector
- Q?: symbol Device:Q_NMOS_DGS -> Milpitas-rescue:Q_NMOS_DGS-Device
- R? (x25): symbol Device:R -> Milpitas-rescue:R-Device
- SW? (x2): symbol Switch:SW_SPST -> Milpitas-rescue:SW_SPST-Switch
- TP? (x3): symbol Connector:TestPoint -> Milpitas-rescue:TestPoint-Connector
- U? (x3): symbol hypersymbols:BTS61363DAUMA1 -> Milpitas-rescue:BTS61363DAUMA1-hypersymbols
- U?: symbol hypersymbols:ACS711 -> Milpitas-rescue:ACS711-hypersymbols
- U?: symbol 4xxx:4011 -> Milpitas-rescue:4011-4xxx
- U?: symbol hypersymbols:XTR2005Z -> Milpitas-rescue:XTR2005Z-hypersymbols
- U?: symbol Analog_ADC:ADS1015IDGS -> Milpitas-rescue:ADS1015IDGS-Analog_ADC
- U?: symbol hypersymbols:ISO1541 -> Milpitas-rescue:ISO1541-hypersymbols
- U?: symbol Isolator:SFH617A-3X001 -> Milpitas-rescue:SFH617A-3X001-Isolator
Connections:
- net +5V: no longer R?.1
- net GND: now also R?.2
- net GNDS: no longer C?.1
- net HP_CTL: now also R?.1; no longer R?.2
- net at R?.2, SW?.2 (B), U?.2 (~IN): now also C?.1
Other:
- moved on the sheet: C?, R?
