File: Milpitas/NAP_PoE.sch (KiCad schematic (older format))
At the start: 2 parts

Commit message: Updated some silly mistakes
Updated some silly mistakes,
- capacitor decoupled to gnd
- Added option for jumper control to 2 24V modules
Parts:
- J? (x2): symbol Connector:RJ45 -> Milpitas-rescue:RJ45-Connector
Changed lines of the file:
@@
 EESchema Schematic File Version 4
 LIBS:Milpitas-cache
-EELAYER 26 0
+EELAYER 29 0
 EELAYER END
 $Descr A4 11693 8268
@@
 $EndDescr
 $Comp
-L Connector:RJ45 J?
+L Milpitas-rescue:RJ45-Connector J?
 U 1 1 5E076C78
 P 3750 3600
@@
 $EndComp
 $Comp
-L Connector:RJ45 J?
+L Milpitas-rescue:RJ45-Connector J?
 U 1 1 5E076CC0
 P 5700 3600
@@
 	5150 4000 5150 4300
 $Comp
-L power:GND #PWR?
+L Milpitas-rescue:GND-power #PWR?
 U 1 1 5E07711E
 P 5150 4300
