File: Milpitas/conversionAndIsolation.sch (KiCad schematic (older format))
At the start: 61 parts

Commit message: Updated some silly mistakes
Updated some silly mistakes,
- capacitor decoupled to gnd
- Added option for jumper control to 2 24V modules
Parts:
- added R?: 0, symbol Milpitas-rescue:R-Device
- C? (x21): symbol Device:C_Small -> Milpitas-rescue:C_Small-Device
- C? (x2): symbol Device:CP -> Milpitas-rescue:CP-Device
- D? (x5): symbol Device:LED -> Milpitas-rescue:LED-Device
- R? (x18): symbol Device:R -> Milpitas-rescue:R-Device
- R?: value 4k -> 0; symbol Device:R -> Milpitas-rescue:R-Device
- RV? (x3): symbol Device:R_POT -> Milpitas-rescue:R_POT-Device
- TP? (x4): symbol Connector:TestPoint -> Milpitas-rescue:TestPoint-Connector
- U?: symbol hypersymbols:UEI15-050-Q48N-C -> Milpitas-rescue:UEI15-050-Q48N-C-hypersymbols
- U?: symbol hypersymbols:UWQ-1217-Q48NB-C -> Milpitas-rescue:UWQ-1217-Q48NB-C-hypersymbols
- U? (x2): symbol hypersymbols:V24C24C150BL -> Milpitas-rescue:V24C24C150BL-hypersymbols
- U? (x3): symbol Isolator:SFH617A-3X001 -> Milpitas-rescue:SFH617A-3X001-Isolator
Connections:
- net 24V_CTL: now also R?.1, U?.4, R?.1; no longer R?.2, U?.2 (PC), U?.2 (PC)
- new net 24V_CTL_1: R?.2, U?.2 (PC)
- new net 24V_CTL_2: R?.2, U?.2 (PC)
Other:
- moved on the sheet: R?

Commit message: Updated input control circuitry. Rationale and calcs in google drive.
Updated and added all part numbers for input protection circuitry. Not yet ready for review.
Parts:
- removed R? (x4): 0, symbol Milpitas-rescue:R-Device
- removed R?: R, symbol Milpitas-rescue:R-Device
- removed U? (x3): SFH617A-3X001, Package_DIP:DIP-4_W7.62mm, symbol Milpitas-rescue:SFH617A-3X001-Isolator
- added R? (x6): R, symbol Device:R
Connections:
- net labels added: +12V, +24V, +5V
- net labels removed: +3.3V, 12V_MCU_CTL, 24V_MCU_CTL, 5V_MCU_CTL
- wire segments 196 -> 192
Other:
- note added: "Populate pull up or pull down\nfor default on or off depending\non what module/function is needed."
- note added: "Population options\ndepending on if both modules\nare being used.\n"
- note added: "Pulldown for default off\nuntil driven high.\n"
- note removed: "Pullup on LED side means\noutput signal is default low"
- note removed: "TODO: Add 3.3V LDO for Paraduino"
- moved on the sheet: C?, D?, R?, RV?, TP?, U?
