File: Milpitas/paraduino.sch (KiCad schematic (older format))
At the start: 0 parts

Commit message: Updated input control circuitry. Rationale and calcs in google drive.
Updated and added all part numbers for input protection circuitry. Not yet ready for review.
Parts:
- added J?: Conn_01x04, symbol Connector_Generic:Conn_01x04
- added R? (x5): R, symbol Device:R
- added U?: SMD42, GeneralMCU_Example:SMD42-FTP, symbol GeneralMCU-Example:SMD42
Connections:
- net labels added: +12V, +24V, +3V3, +5V, +BATT, 12V_MCU_CTL, 24V_MCU_CTL, 5V_MCU_CTL, CAN_N, CAN_P, CAN_SHIELD, GND, HP_CTL, i_csense, i_vsense, o12_csense, o24_csense, o5_csense
- wire segments 0 -> 38
- no-connect marks 0 -> 1
Other:
- note added: "Name change for Diff routing\nCAN_N = CAN_L\nCAN_H = CAN_P"
- note added: "ONLY POPULATE ONE AT A TIME\n"
