File: BigSur/PumpDrivers.sch (KiCad schematic (older format))
At the start: 6 parts, among them Q1 TSM900N10, Q2 TSM900N10

Commit message: Added mounting holes, CAN connector,  indicator LEDs, started general purpose relays
Parts:
- removed D3, D4: NTS12120EMFST1G, BigSur:ONSemi_SMD_Schottky_NTS12120EMFS, symbol Device:D_Schottky
- removed Q1, Q2: TSM900N10, Package_TO_SOT_SMD:TO-252-2, symbol Device:Q_NMOS_GDS
- removed R11, R12: 100K, Resistor_SMD:R_0603_1608Metric_Pad1.05x0.95mm_HandSolder, symbol Device:R_US
Changed lines of the file:
@@
 EESchema Schematic File Version 4
 LIBS:BigSur-cache
-EELAYER 29 0
+EELAYER 30 0
 EELAYER END
 $Descr A4 11693 8268
@@
 Comment4 "Jasper Rubin"
 $EndDescr
-$Comp
-L Device:Q_NMOS_GDS Q1
-U 1 1 5D7D3E10
-P 2400 1900
-F 0 "Q1" H 2606 1946 50  0000 L CNN
-F 1 "TSM900N10" H 2606 1855 50  0000 L CNN
-F 2 "Package_TO_SOT_SMD:TO-252-2" H 2600 2000 50  0001 C CNN
-F 3 "https://www.taiwansemi.com/products/datasheet/TSM900N10_A15.pdf" H 2400 1900 50  0001 C CNN
-F 4 "https://www.digikey.ca/product-detail/en/taiwan-semiconductor-corporation/TSM900N10CP-ROG/TSM900N10CPROGCT-ND/7360607" H 2400 1900 50  0001 C CNN "Digikey"
-	1    2400 1900
-	1    0    0    -1
-$EndComp
-Wire Wire Line
-	2500 2100 2500 2350
-$Comp
-L power:GND #PWR042
-U 1 1 5D7D4C28
-P 2500 2350
-F 0 "#PWR042" H 2500 2100 50  0001 C CNN
-F 1 "GND" H 2505 2177 50  0000 C CNN
-F 2 "" H 2500 2350 50  0001 C CNN
-F 3 "" H 2500 2350 50  0001 C CNN
-	1    2500 2350
-	1    0    0    -1
-$EndComp
-Wire Wire Line
-	2500 1700 2500 1600
-Wire Wire Line
-	2500 1600 2650 1600
-Text GLabel 2650 1600 2    50   BiDi ~ 0
-PUMP_LS_CHANNEL_1
-Connection ~ 2500 1600
-Wire Wire Line
-	2200 1900 2000 1900
-Wire Wire Line
-	2000 1900 2000 1950
-Connection ~ 2000 1900
-Wire Wire Line
-	2000 1900 1700 1900
-$Comp
-L Device:R_US R11
-U 1 1 5D7D75FE
-P 2000 2100
-F 0 "R11" H 2068 2146 50  0000 L CNN
-F 1 "100K" H 2068 2055 50  0000 L CNN
-F 2 "Resistor_SMD:R_0603_1608Metric_Pad1.05x0.95mm_HandSolder" V 2040 2090 50  0001 C CNN
-F 3 "~" H 2000 2100 50  0001 C CNN
-	1    2000 2100
-	1    0    0    -1
-$EndComp
-$Comp
-L power:GND #PWR041
-U 1 1 5D7D85EE
-P 2000 2350
-F 0 "#PWR041" H 2000 2100 50  0001 C CNN
-F 1 "GND" H 2005 2177 50  0000 C CNN
-F 2 "" H 2000 2350 50  0001 C CNN
-F 3 "" H 2000 2350 50  0001 C CNN
-	1    2000 2350
-	1    0    0    -1
-$EndComp
-Wire Wire Line
-	2000 2350 2000 2250
-Wire Wire Line
-	2500 1550 2500 1600
-$Comp
-L power:+24V #PWR040
-U 1 1 5D6DC51E
-P 2500 1150
-F 0 "#PWR040" H 2500 1000 50  0001 C CNN
-F 1 "+24V" H 2515 1323 50  0000 C CNN
-F 2 "" H 2500 1150 50  0001 C CNN
-F 3 "" H 2500 1150 50  0001 C CNN
-	1    2500 1150
-	1    0    0    -1
-$EndComp
-$Comp
-L Device:D_Schottky D3
-U 1 1 5D6DD7E1
-P 2500 1400
-F 0 "D3" V 2454 1479 50  0000 L CNN
-F 1 "NTS12120EMFST1G" V 2545 1479 50  0000 L CNN
-F 2 "BigSur:ONSemi_SMD_Schottky_NTS12120EMFS" H 2500 1400 50  0001 C CNN
-F 3 "https://www.onsemi.com/pub/Collateral/NTS12120EMFS-D.PDF" H 2500 1400 50  0001 C CNN
-F 4 "https://www.digikey.ca/product-detail/en/on-semiconductor/NTS12120EMFST1G/NTS12120EMFST1GOSCT-ND/8538813" V 2500 1400 50  0001 C CNN "Digikey"
-	1    2500 1400
-	0    1    1    0
-$EndComp
-Wire Wire Line
-	2500 1150 2500 1250
-Text GLabel 1700 1900 0    50   BiDi ~ 0
-PUMP_INPUT_1
-$Comp
-L Device:Q_NMOS_GDS Q2
-U 1 1 5D85B099
-P 2400 3700
-F 0 "Q2" H 2606 3746 50  0000 L CNN
-F 1 "TSM900N10" H 2606 3655 50  0000 L CNN
-F 2 "Package_TO_SOT_SMD:TO-252-2" H 2600 3800 50  0001 C CNN
-F 3 "https://www.taiwansemi.com/products/datasheet/TSM900N10_A15.pdf" H 2400 3700 50  0001 C CNN
-F 4 "https://www.digikey.ca/product-detail/en/taiwan-semiconductor-corporation/TSM900N10CP-ROG/TSM900N10CPROGCT-ND/7360607" H 2400 3700 50  0001 C CNN "Digikey"
-	1    2400 3700
-	1    0    0    -1
-$EndComp
-Wire Wire Line
-	2500 3900 2500 4150
-$Comp
-L power:GND #PWR045
-U 1 1 5D85B0A4
-P 2500 4150
-F 0 "#PWR045" H 2500 3900 50  0001 C CNN
-F 1 "GND" H 2505 3977 50  0000 C CNN
-F 2 "" H 2500 4150 50  0001 C CNN
-F 3 "" H 2500 4150 50  0001 C CNN
-	1    2500 4150
-	1    0    0    -1
-$EndComp
-Wire Wire Line
-	2500 3500 2500 3400
-Wire Wire Line
-	2500 3400 2650 3400
-Text GLabel 2650 3400 2    50   BiDi ~ 0
-PUMP_LS_CHANNEL_2
-Connection ~ 2500 3400
-Wire Wire Line
-	2200 3700 2000 3700
-Wire Wire Line
-	2000 3700 2000 3750
-Connection ~ 2000 3700
-Wire Wire Line
-	2000 3700 1700 3700
-$Comp
-L Device:R_US R12
-U 1 1 5D85B0B6
-P 2000 3900
-F 0 "R12" H 2068 3946 50  0000 L CNN
-F 1 "100K" H 2068 3855 50  0000 L CNN
-F 2 "Resistor_SMD:R_0603_1608Metric_Pad1.05x0.95mm_HandSolder" V 2040 3890 50  0001 C CNN
-F 3 "~" H 2000 3900 50  0001 C CNN
-	1    2000 3900
-	1    0    0    -1
-$EndComp
-$Comp
-L power:GND #PWR044
-U 1 1 5D85B0C0
-P 2000 4150
-F 0 "#PWR044" H 2000 3900 50  0001 C CNN
-F 1 "GND" H 2005 3977 50  0000 C CNN
-F 2 "" H 2000 4150 50  0001 C CNN
-F 3 "" H 2000 4150 50  0001 C CNN
-	1    2000 4150
-	1    0    0    -1
-$EndComp
-Wire Wire Line
-	2000 4150 2000 4050
-Wire Wire Line
-	2500 3350 2500 3400
-$Comp
-L power:+24V #PWR043
-U 1 1 5D85B0CC
-P 2500 2950
-F 0 "#PWR043" H 2500 2800 50  0001 C CNN
-F 1 "+24V" H 2515 3123 50  0000 C CNN
-F 2 "" H 2500 2950 50  0001 C CNN
-F 3 "" H 2500 2950 50  0001 C CNN
-	1    2500 2950
-	1    0    0    -1
-$EndComp
-$Comp
-L Device:D_Schottky D4
-U 1 1 5D85B0D7
-P 2500 3200
-F 0 "D4" V 2454 3279 50  0000 L CNN
-F 1 "NTS12120EMFST1G" V 2545 3279 50  0000 L CNN
-F 2 "BigSur:ONSemi_SMD_Schottky_NTS12120EMFS" H 2500 3200 50  0001 C CNN
-F 3 "https://www.onsemi.com/pub/Collateral/NTS12120EMFS-D.PDF" H 2500 3200 50  0001 C CNN
-F 4 "https://www.digikey.ca/product-detail/en/on-semiconductor/NTS12120EMFST1G/NTS12120EMFST1GOSCT-ND/8538813" V 2500 3200 50  0001 C CNN "Digikey"
-	1    2500 3200
-	0    1    1    0
-$EndComp
-Wire Wire Line
-	2500 2950 2500 3050
-Text GLabel 1700 3700 0    50   BiDi ~ 0
-PUMP_INPUT_2
 $EndSCHEMATC
