File: BigSur/BigSur.kicad_pcb (KiCad board)
At the start: 2 copper layers, 123.5 x 131.5 mm, 148 parts, among them J1 XT30PW-M, J10 XT30PW-M, J12 XT30PW-M, J14 XT30PW-M, J15 XT30PW-M, J16 XT30PW-M, J2 XT30PW-M, J3 XT30PW-M, J4 XT30PW-M, J5 XT30PW-M, J6 XT30PW-M, J7 XT30PW-M, J8 XT30PW-M, J9 XT30PW-M, K1 G5LE-1A-VDDC12, K2 G5LE-1A-VDDC12, K3 G5LE-1A-VDDC12, K4 G5LE-1A-VDDC12, Q1 TSM900N10, Q2 TSM900N10, Q3 MMBT3904-7-F, Q4 MMBT3904-7-F, Q5 MMBT3904-7-F, Q6 MMBT3904-7-F, U1 DRV103H, U10 MCP6L02T-E_MS, U11 74LVC1G08W5-7, U12 ACS70331EESATR-2P5U3, U2 DRV103H, U3 DRV8806, U4 SMD46, U5 ACS70331EESATR-2P5U3, U6 ACS70331EESATR-2P5U3, U7 ACS70331EESATR-2P5U3, U8 ACS70331EESATR-2P5U3, U9 ACS70331EESATR-2P5U3

Commit message: More layout changes
Parts:
- C30, C34, C35, D22, R37, R39, R40, R41, U10: moved to B.Cu
- R15: moved to F.Cu
- moved D22 47.6 mm to (115.3, 45.4), turned to 90 degrees
- moved R37 47.6 mm to (118.8, 45.4), turned to 90 degrees
- moved C34 37.6 mm to (115.3, 50.4), turned to 90 degrees
- moved R39 37.6 mm to (118.3, 50.4), turned to 270 degrees
- moved U11 36.0 mm to (127.0, 52.1), turned to 90 degrees
- moved U10 33.6 mm to (121.3, 52.4), turned to 90 degrees
- moved C30 29.6 mm to (115.3, 54.4), turned to 270 degrees
- moved R40 29.3 mm to (118.3, 54.6), turned to 270 degrees
- moved C10 26.2 mm to (111.8, 79.0)
- moved C11 26.2 mm to (111.8, 74.0)
- moved C12 26.2 mm to (117.8, 95.5)
- moved C13 26.2 mm to (117.8, 90.5)
- moved C14 26.2 mm to (117.8, 85.5)
- moved C15 26.2 mm to (117.8, 80.5)
- moved C16 26.2 mm to (117.8, 75.5)
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