File: GeneralMCU/noncast_temp_pcbs/GeneralMCU.kicad_pcb (KiCad board)
At the start: 2 copper layers, 30 x 80 mm, 97 parts, among them J1 ARM_JTAG_SWD, J2 SMD46 castellation PKG, J3 USB_B_Micro, J5 PWR, J6 OLED, Q1 Q_NMOS_DGS, SW1 USER, SW2 RESET, U1 STM32F303R6Tx, U2 SN65HVD230, U3 AZ1117-3.3, U4 P78E05-1000, U5 DS18B20, Y1 32.768kHz, Y2 8MHz

Commit message: Adding in old rescued folder.
Parts:
- removed J6: OLED, µ104KiCAD:I2C_OLED
Routing:
- net /I2C1_SDA: track 41.9 -> 31.4 mm, vias 8 -> 7
- net /I2C1_SCL: track 36.4 -> 31.9 mm, vias 9 -> 7
- net GND: track 134.7 -> 133.1 mm
- net +5V: track 147.7 -> 149.1 mm, vias 11 -> 12
- net +V: track 57.6 -> 58.9 mm, vias 3 -> 4
- net +3V3: track 145.7 -> 146.9 mm, vias 7 -> 8
- net /PC1: track 16.2 -> 15.6 mm
