File: Milpitas_BMS/_autosave-Milpitas_BMS.kicad_pcb (KiCad board)
At the start: 2 copper layers, 333 parts, among them J100 JTAG, J102 CAN_CONN, J102 DIAGS_CON, J104 CAN_CONN, J400 CHG INPUT, J401 POWER_OUTPUT, J402 BATT_PWR_INPUT, J500 SOUTH CELL CONN, J501 NORTH CELL CONN, Q400 RU1J002YNTCL, Q401 RU1J002YNTCL, Q402 RU1J002YNTCL, SW100 SW_SPST, SW101 SW_SPST, U1 BQ79606, U100 MIC5283-3.3ML-TR, U101 STM32F303RETx, U102 SN65HVD232, U200 BQ79606, U400 ACS711, U401 BTS6163DAUMA1, U402 ACS711, U403 BTS6163DAUMA1, U404 BTS6163DAUMA1, U405 ACS711, Y1 32.768kHz, Y2 32MHz

Commit message: For review call
Parts:
- moved H0 300.6 mm to (307.7, -1.70)
- moved H1 300.6 mm to (307.7, -8.65)
- moved H2 300.6 mm to (300.8, -1.70)
- moved H3 300.6 mm to (300.8, -8.65)
- moved R1 300.6 mm to (317.2, -7.58)
- moved R2 300.6 mm to (313.2, -2.56)
- moved R3 300.6 mm to (313.2, -0.05)
- moved R4 300.6 mm to (317.2, -5.07)
- moved R5 300.6 mm to (321.2, -7.58)
- moved R6 300.6 mm to (313.2, -7.58)
- moved R7 300.6 mm to (317.2, -2.56)
- moved R8 300.6 mm to (317.2, -0.05)
- moved R210 104.2 mm to (35.6, 59.9)
- moved R203 104.1 mm to (35.6, 61.5)
- moved R202 104.1 mm to (35.6, 55.4)
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Other:
- copper layers 2 -> 4
