File: Milpitas_BMS/Milpitas_BMS.sch (KiCad schematic (older format))
At the start: 12 parts

Commit message: updated some parts to inclued footprints + digikey P/N
Parts:
- H0, H1, H2, H3: footprint (none) -> MountingHole:MountingHole_3.2mm_M3_Pad_Via
- R1, R2, R3, R4, R5, R6, R7, R8: footprint (none) -> Resistor_SMD:R_0603_1608Metric
Changed lines of the file:
@@
 F 0 "H0" H 9100 5649 50  0000 L CNN
 F 1 "TL" H 9100 5558 50  0000 L CNN
-F 2 "" H 9000 5600 50  0001 C CNN
+F 2 "MountingHole:MountingHole_3.2mm_M3_Pad_Via" H 9000 5600 50  0001 C CNN
 F 3 "~" H 9000 5600 50  0001 C CNN
 	1    9000 5600
@@
 F 0 "H1" H 9750 5649 50  0000 L CNN
 F 1 "TR" H 9750 5558 50  0000 L CNN
-F 2 "" H 9650 5600 50  0001 C CNN
+F 2 "MountingHole:MountingHole_3.2mm_M3_Pad_Via" H 9650 5600 50  0001 C CNN
 F 3 "~" H 9650 5600 50  0001 C CNN
 	1    9650 5600
@@
 F 0 "H2" H 10350 5649 50  0000 L CNN
 F 1 "BL" H 10350 5558 50  0000 L CNN
-F 2 "" H 10250 5600 50  0001 C CNN
+F 2 "MountingHole:MountingHole_3.2mm_M3_Pad_Via" H 10250 5600 50  0001 C CNN
 F 3 "~" H 10250 5600 50  0001 C CNN
 	1    10250 5600
@@
 F 0 "H3" H 10950 5649 50  0000 L CNN
 F 1 "BR" H 10950 5558 50  0000 L CNN
-F 2 "" H 10850 5600 50  0001 C CNN
+F 2 "MountingHole:MountingHole_3.2mm_M3_Pad_Via" H 10850 5600 50  0001 C CNN
 F 3 "~" H 10850 5600 50  0001 C CNN
 	1    10850 5600
@@
 F 0 "R1" H 8750 6000 50  0000 L CNN
 F 1 "0" H 8800 5900 50  0000 L CNN
-F 2 "" V 8830 5950 50  0001 C CNN
+F 2 "Resistor_SMD:R_0603_1608Metric" V 8830 5950 50  0001 C CNN
 F 3 "~" H 8900 5950 50  0001 C CNN
 	1    8900 5950
@@
 F 0 "R2" H 9170 5996 50  0000 L CNN
 F 1 "0" H 9170 5905 50  0000 L CNN
-F 2 "" V 9030 5950 50  0001 C CNN
+F 2 "Resistor_SMD:R_0603_1608Metric" V 9030 5950 50  0001 C CNN
 F 3 "~" H 9100 5950 50  0001 C CNN
 	1    9100 5950
@@
 $EndComp
 $Comp
-L power:GND #PWR?
+L power:GND #PWR0101
 U 1 1 62653353
 P 9000 6250
-F 0 "#PWR?" H 9000 6000 50  0001 C CNN
+F 0 "#PWR0101" H 9000 6000 50  0001 C CNN
 F 1 "GND" H 9005 6077 50  0000 C CNN
 F 2 "" H 9000 6250 50  0001 C CNN
@@
 F 0 "R3" H 9400 6000 50  0000 L CNN
 F 1 "0" H 9450 5900 50  0000 L CNN
-F 2 "" V 9480 5950 50  0001 C CNN
+F 2 "Resistor_SMD:R_0603_1608Metric" V 9480 5950 50  0001 C CNN
 F 3 "~" H 9550 5950 50  0001 C CNN
 	1    9550 5950
@@
 F 0 "R4" H 9820 5996 50  0000 L CNN
 F 1 "0" H 9820 5905 50  0000 L CNN
-F 2 "" V 9680 5950 50  0001 C CNN
+F 2 "Resistor_SMD:R_0603_1608Metric" V 9680 5950 50  0001 C CNN
 F 3 "~" H 9750 5950 50  0001 C CNN
 	1    9750 5950
@@
 $EndComp
 $Comp
-L power:GND #PWR?
+L power:GND #PWR0102
 U 1 1 62656DB4
 P 9650 6250
-F 0 "#PWR?" H 9650 6000 50  0001 C CNN
+F 0 "#PWR0102" H 9650 6000 50  0001 C CNN
 F 1 "GND" H 9655 6077 50  0000 C CNN
 F 2 "" H 9650 6250 50  0001 C CNN
@@
 F 0 "R5" H 10000 6000 50  0000 L CNN
 F 1 "0" H 10050 5900 50  0000 L CNN
-F 2 "" V 10080 5950 50  0001 C CNN
+F 2 "Resistor_SMD:R_0603_1608Metric" V 10080 5950 50  0001 C CNN
 F 3 "~" H 10150 5950 50  0001 C CNN
 	1    10150 5950
@@
 F 0 "R6" H 10420 5996 50  0000 L CNN
 F 1 "0" H 10420 5905 50  0000 L CNN
-F 2 "" V 10280 5950 50  0001 C CNN
+F 2 "Resistor_SMD:R_0603_1608Metric" V 10280 5950 50  0001 C CNN
 F 3 "~" H 10350 5950 50  0001 C CNN
 	1    10350 5950
@@
 $EndComp
 $Comp
-L power:GND #PWR?
+L power:GND #PWR0103
 U 1 1 62657F41
 P 10250 6250
-F 0 "#PWR?" H 10250 6000 50  0001 C CNN
+F 0 "#PWR0103" H 10250 6000 50  0001 C CNN
 F 1 "GND" H 10255 6077 50  0000 C CNN
 F 2 "" H 10250 6250 50  0001 C CNN
@@
 F 0 "R7" H 10600 6000 50  0000 L CNN
 F 1 "0" H 10650 5900 50  0000 L CNN
-F 2 "" V 10680 5950 50  0001 C CNN
+F 2 "Resistor_SMD:R_0603_1608Metric" V 10680 5950 50  0001 C CNN
 F 3 "~" H 10750 5950 50  0001 C CNN
 	1    10750 5950
@@
 F 0 "R8" H 11020 5996 50  0000 L CNN
 F 1 "0" H 11020 5905 50  0000 L CNN
-F 2 "" V 10880 5950 50  0001 C CNN
+F 2 "Resistor_SMD:R_0603_1608Metric" V 10880 5950 50  0001 C CNN
 F 3 "~" H 10950 5950 50  0001 C CNN
 	1    10950 5950
@@
 $EndComp
 $Comp
-L power:GND #PWR?
+L power:GND #PWR0104
 U 1 1 62659BFA
 P 10850 6250
-F 0 "#PWR?" H 10850 6000 50  0001 C CNN
+F 0 "#PWR0104" H 10850 6000 50  0001 C CNN
 F 1 "GND" H 10855 6077 50  0000 C CNN
 F 2 "" H 10850 6250 50  0001 C CNN
@@
 Data
 89 50 4E 47 0D 0A 1A 0A 00 00 00 0D 49 48 44 52 00 00 00 54 00 00 00 4E 08 02 00 00 00 31 44 A6
-6B 00 00 00 03 73 42 49 54 08 08 08 DB E1 4F E0 00 00 00 09 70 48 59 73 00 00 2E 23 00 00 2E 23
-01 78 A5 3F 76 00 00 12 2F 49 44 41 54 78 9C E5 5C 5B 6C 54 C5 1B 9F 99 33 E7 EC AD 2D 2D 17 01
+6B 00 00 00 03 73 42 49 54 08 08 08 DB E1 4F E0 00 00 00 09 70 48 59 73 00 00 2E 18 00 00 2E 18
+01 2A AA 27 20 00 00 12 2F 49 44 41 54 78 9C E5 5C 5B 6C 54 C5 1B 9F 99 33 E7 EC AD 2D 2D 17 01
 83 12 51 63 D4 48 31 48 22 F5 C5 27 20 91 10 13 63 44 02 94 B2 B8 40 5B 50 44 A3 0F 62 E2 93 04
 13 49 0A 85 82 6D 90 18 11 8C 25 10 5E 10 89 BC 98 A8 58 8D 97 68 8A 26 6A 82 4A E4 56 DA 2E 7B
@@
 Data
 89 50 4E 47 0D 0A 1A 0A 00 00 00 0D 49 48 44 52 00 00 00 54 00 00 00 4E 08 02 00 00 00 31 44 A6
-6B 00 00 00 03 73 42 49 54 08 08 08 DB E1 4F E0 00 00 00 09 70 48 59 73 00 00 2E 23 00 00 2E 23
-01 78 A5 3F 76 00 00 12 2F 49 44 41 54 78 9C E5 5C 5B 6C 54 C5 1B 9F 99 33 E7 EC AD 2D 2D 17 01
+6B 00 00 00 03 73 42 49 54 08 08 08 DB E1 4F E0 00 00 00 09 70 48 59 73 00 00 2E 18 00 00 2E 18
+01 2A AA 27 20 00 00 12 2F 49 44 41 54 78 9C E5 5C 5B 6C 54 C5 1B 9F 99 33 E7 EC AD 2D 2D 17 01
 83 12 51 63 D4 48 31 48 22 F5 C5 27 20 91 10 13 63 44 02 94 B2 B8 40 5B 50 44 A3 0F 62 E2 93 04
 13 49 0A 85 82 6D 90 18 11 8C 25 10 5E 10 89 BC 98 A8 58 8D 97 68 8A 26 6A 82 4A E4 56 DA 2E 7B
@@
 Data
 89 50 4E 47 0D 0A 1A 0A 00 00 00 0D 49 48 44 52 00 00 00 54 00 00 00 4E 08 02 00 00 00 31 44 A6
-6B 00 00 00 03 73 42 49 54 08 08 08 DB E1 4F E0 00 00 00 09 70 48 59 73 00 00 2E 23 00 00 2E 23
-01 78 A5 3F 76 00 00 12 2F 49 44 41 54 78 9C E5 5C 5B 6C 54 C5 1B 9F 99 33 E7 EC AD 2D 2D 17 01
+6B 00 00 00 03 73 42 49 54 08 08 08 DB E1 4F E0 00 00 00 09 70 48 59 73 00 00 2E 18 00 00 2E 18
+01 2A AA 27 20 00 00 12 2F 49 44 41 54 78 9C E5 5C 5B 6C 54 C5 1B 9F 99 33 E7 EC AD 2D 2D 17 01
 83 12 51 63 D4 48 31 48 22 F5 C5 27 20 91 10 13 63 44 02 94 B2 B8 40 5B 50 44 A3 0F 62 E2 93 04
 13 49 0A 85 82 6D 90 18 11 8C 25 10 5E 10 89 BC 98 A8 58 8D 97 68 8A 26 6A 82 4A E4 56 DA 2E 7B
@@
 Data
 89 50 4E 47 0D 0A 1A 0A 00 00 00 0D 49 48 44 52 00 00 00 54 00 00 00 4E 08 02 00 00 00 31 44 A6
-6B 00 00 00 03 73 42 49 54 08 08 08 DB E1 4F E0 00 00 00 09 70 48 59 73 00 00 2E 23 00 00 2E 23
-01 78 A5 3F 76 00 00 12 2F 49 44 41 54 78 9C E5 5C 5B 6C 54 C5 1B 9F 99 33 E7 EC AD 2D 2D 17 01
+6B 00 00 00 03 73 42 49 54 08 08 08 DB E1 4F E0 00 00 00 09 70 48 59 73 00 00 2E 18 00 00 2E 18
+01 2A AA 27 20 00 00 12 2F 49 44 41 54 78 9C E5 5C 5B 6C 54 C5 1B 9F 99 33 E7 EC AD 2D 2D 17 01
 83 12 51 63 D4 48 31 48 22 F5 C5 27 20 91 10 13 63 44 02 94 B2 B8 40 5B 50 44 A3 0F 62 E2 93 04
 13 49 0A 85 82 6D 90 18 11 8C 25 10 5E 10 89 BC 98 A8 58 8D 97 68 8A 26 6A 82 4A E4 56 DA 2E 7B
@@
 Data
 89 50 4E 47 0D 0A 1A 0A 00 00 00 0D 49 48 44 52 00 00 00 54 00 00 00 4E 08 02 00 00 00 31 44 A6
-6B 00 00 00 03 73 42 49 54 08 08 08 DB E1 4F E0 00 00 00 09 70 48 59 73 00 00 2E 23 00 00 2E 23
-01 78 A5 3F 76 00 00 12 2F 49 44 41 54 78 9C E5 5C 5B 6C 54 C5 1B 9F 99 33 E7 EC AD 2D 2D 17 01
+6B 00 00 00 03 73 42 49 54 08 08 08 DB E1 4F E0 00 00 00 09 70 48 59 73 00 00 2E 18 00 00 2E 18
+01 2A AA 27 20 00 00 12 2F 49 44 41 54 78 9C E5 5C 5B 6C 54 C5 1B 9F 99 33 E7 EC AD 2D 2D 17 01
 83 12 51 63 D4 48 31 48 22 F5 C5 27 20 91 10 13 63 44 02 94 B2 B8 40 5B 50 44 A3 0F 62 E2 93 04
 13 49 0A 85 82 6D 90 18 11 8C 25 10 5E 10 89 BC 98 A8 58 8D 97 68 8A 26 6A 82 4A E4 56 DA 2E 7B
@@
 Data
 89 50 4E 47 0D 0A 1A 0A 00 00 00 0D 49 48 44 52 00 00 00 54 00 00 00 4E 08 02 00 00 00 31 44 A6
-6B 00 00 00 03 73 42 49 54 08 08 08 DB E1 4F E0 00 00 00 09 70 48 59 73 00 00 2E 23 00 00 2E 23
-01 78 A5 3F 76 00 00 12 2F 49 44 41 54 78 9C E5 5C 5B 6C 54 C5 1B 9F 99 33 E7 EC AD 2D 2D 17 01
+6B 00 00 00 03 73 42 49 54 08 08 08 DB E1 4F E0 00 00 00 09 70 48 59 73 00 00 2E 18 00 00 2E 18
+01 2A AA 27 20 00 00 12 2F 49 44 41 54 78 9C E5 5C 5B 6C 54 C5 1B 9F 99 33 E7 EC AD 2D 2D 17 01
 83 12 51 63 D4 48 31 48 22 F5 C5 27 20 91 10 13 63 44 02 94 B2 B8 40 5B 50 44 A3 0F 62 E2 93 04
 13 49 0A 85 82 6D 90 18 11 8C 25 10 5E 10 89 BC 98 A8 58 8D 97 68 8A 26 6A 82 4A E4 56 DA 2E 7B

Commit message: lots of little fixes
Parts:
- added C1: CXX, Capacitor_SMD:C_0603_1608Metric, symbol Device:C_Small
- added FB1: Choke, symbol Device:Ferrite_Bead_Small
- added TP2: N_GND, Resistor_SMD:R_1206_3216Metric, symbol Connector:TestPoint
- added TP3: GND, Resistor_SMD:R_1206_3216Metric, symbol Connector:TestPoint
- H0, H1, H2, H3: footprint MountingHole:MountingHole_3.2mm_M3_Pad_Via -> MountingHole:MountingHole_2.7mm_M2.5_Pad_Via
Connections:
- net GND: now also C1.1, FB1.1, TP3.1
- new net GNDS: C1.2, FB1.2, TP2.1
- no-connect marks 0 -> 2
Other:
- note added: "Options for ground \ncoupling (DNC)"
- moved on the sheet: H0, H1, H2, H3, R1, R2, R3, R4, R5, R6, R7, R8

Commit message: (maybe) final placement V1,0
Changed lines of the file:
@@
 Wire Bus Line
 	7050 5350 7700 5350
-Text Label 3600 4600 0    39   ~ 0
-A[0..12]
 $EndSCHEMATC
