File: Milpitas_BMS/Milpitas_BMS.kicad_pcb (KiCad board)
At the start: 2 copper layers, 298 parts, among them J100 JTAG, J102 CAN_CONN, J3 CAN_CONN, Q400 RU1J002YNTCL, Q401 RU1J002YNTCL, Q402 RU1J002YNTCL, U1 BQ79606, U100 MIC5283-3.3ML-TR, U101 STM32F303RETx, U102 SN65HVD232, U200 BQ79606, U400 ACS711, U401 BTS6163DAUMA1, U402 ACS711, U403 BTS6163DAUMA1, U404 BTS6163DAUMA1, U405 ACS711

Commit message: lots of little fixes
Parts:
- added C1: CXX, Capacitor_SMD:C_0603_1608Metric, F.Cu at (27.9, 89.5)
- added C111: 7pF, Capacitor_SMD:C_0603_1608Metric, F.Cu at (318.8, 61.9)
- added C112: 7pF, Capacitor_SMD:C_0603_1608Metric, F.Cu at (317.5, 66.9)
- added C113: 8pF, Capacitor_SMD:C_0603_1608Metric, F.Cu at (335.5, 49.4)
- added C114: 8pF, Capacitor_SMD:C_0603_1608Metric, F.Cu at (335.5, 46.8)
- added D101: D_Zener, Diode_SMD:D_SOD-323F, F.Cu at (306.6, 62.6)
- added D102: D_Zener, Diode_SMD:D_SOD-323F, F.Cu at (318.1, 50.7)
- added D103: D_Zener, Diode_SMD:D_SOD-323F, F.Cu at (316.9, 54.2)
- added D2: D_Zener, Diode_SMD:D_SOD-323F, F.Cu at (296.6, 69.5)
- added J400: CHG INPUT, Milpitas_BMS:XT30-RIGHT-ANGLE, F.Cu at (275.1, 128.3)
- added J401: POWER_OUTPUT, Milpitas_BMS:XT30-RIGHT-ANGLE, F.Cu at (275.2, 111.5)
- added J402: BATT_PWR_INPUT, Milpitas_BMS:XT30-RIGHT-ANGLE, F.Cu at (265.9, 155.7)
- added J500: SOUTH CELL CONN, Connector_Molex:Molex_Micro-Fit_3.0_43045-2000_2x10_P3.00mm_Horizontal, F.Cu at (130.0, 71.1)
- added J501: NORTH CELL CONN, Connector_Molex:Molex_Micro-Fit_3.0_43045-2000_2x10_P3.00mm_Horizontal, F.Cu at (128.8, 133.9)
- added R10: 0, Resistor_SMD:R_0603_1608Metric, F.Cu at (331.5, 49.4)
- added R124: 10k, Resistor_SMD:R_0603_1608Metric, F.Cu at (304.8, 70.5)
- added R125: 10k, Resistor_SMD:R_0603_1608Metric, F.Cu at (322.8, 59.5)
- added R9: 0, Resistor_SMD:R_0603_1608Metric, F.Cu at (309.4, 65.4)
- added SW100: SW_SPST, Milpitas_BMS:KSR223GLFG, F.Cu at (298.0, 43.0)
- added SW101: SW_SPST, Milpitas_BMS:KSR223GLFG, F.Cu at (283.6, 57.5)
- added TP2: N_GND, Resistor_SMD:R_1206_3216Metric, F.Cu at (145.3, 138.8)
- added TP3: GND, Resistor_SMD:R_1206_3216Metric, F.Cu at (28.7, 84.1)
- added Y1: 32.768kHz, Milpitas_BMS:FC-135, F.Cu at (290.7, 69.6)
- added Y2: 32MHz, Milpitas_BMS:NX5032GA, F.Cu at (295.9, 56.8)
- H0, H1, H2, H3: footprint MountingHole:MountingHole_3.2mm_M3_Pad_Via -> MountingHole:MountingHole_2.7mm_M2.5_Pad_Via
- J3: value CAN_CONN -> DIAGS_CON
- moved H2 193.4 mm to (15.4, 92.9)
- moved R2 191.4 mm to (27.9, 92.1)
- moved R7 191.4 mm to (31.9, 92.1)
- moved R3 187.5 mm to (27.9, 94.6)
- moved R8 186.9 mm to (31.9, 94.6)
- moved R4 186.4 mm to (31.9, 89.5)
- moved R6 185.0 mm to (27.9, 87.0)
- moved H1 183.8 mm to (22.4, 86.0)
- moved H3 182.8 mm to (15.4, 86.0)
- moved R1 182.5 mm to (31.9, 87.0)
- moved H0 178.9 mm to (22.4, 92.9)
- moved D105 178.2 mm to (328.5, 41.8)
- moved R5 177.6 mm to (35.9, 87.0)
- moved F400 174.0 mm to (317.2, 114.9)
- moved U404 168.0 mm to (308.3, 117.3)
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Connections:
- net /MCU/BATT_ON renamed /MCU/A11
- net /MCU/CAN_RX_N renamed Net-(R10-Pad2)
- net /MCU/CAN_TX_P renamed Net-(R9-Pad2)
- net /MCU/CHG_ON renamed /MCU/A9
- net /MCU/DIS_ON renamed /MCU/A7
- net /MCU/I_BATT renamed /MCU/A5
- net /MCU/I_CHG renamed /MCU/A3
- net /MCU/I_DIS renamed /MCU/A1
- net /MCU/V_BATT renamed /MCU/A4
- net /MCU/V_CHG renamed /MCU/A6
- net /MCU/V_DIS renamed /MCU/A2
- net /NORTH_BQ/NORTH_CELL0 renamed NORTH_CELL_0
- net /NORTH_BQ/NORTH_CELL2 renamed NORTH_CELL_2
- net /NORTH_BQ/NORTH_CELL3 renamed NORTH_CELL_3
- net /NORTH_BQ/NORTH_CELL6 renamed NORTH_CELL_6
- net /NORTH_BQ/NORTH_THERM1_N renamed NORTH_THERM1_N
- net /NORTH_BQ/NORTH_THERM2_N renamed NORTH_THERM2_N
- net /NORTH_BQ/NORTH_THERM3_N renamed NORTH_THERM3_N
- net /NORTH_BQ/NORTH_THERM4_N renamed NORTH_THERM4_N
- net /NORTH_BQ/NORTH_THERM5_N renamed NORTH_THERM5_N
- net /NORTH_BQ/NORTH_THERM6_N renamed NORTH_THERM6_N
- net /South(Master)_BQ/SOUTH_CELL0 renamed SOUTH_CELL_0
- net /South(Master)_BQ/SOUTH_CELL2 renamed SOUTH_CELL_2
- net /South(Master)_BQ/SOUTH_CELL3 renamed SOUTH_CELL_3
- net /South(Master)_BQ/SOUTH_CELL6 renamed SOUTH_CELL_6
- net /South(Master)_BQ/SOUTH_THERM1_N renamed SOUTH_THERM1_N
- net /South(Master)_BQ/SOUTH_THERM2_N renamed SOUTH_THERM2_N
- net /South(Master)_BQ/SOUTH_THERM3_N renamed SOUTH_THERM3_N
- net /South(Master)_BQ/SOUTH_THERM4_N renamed SOUTH_THERM4_N
- net /South(Master)_BQ/SOUTH_THERM5_N renamed SOUTH_THERM5_N
- net /South(Master)_BQ/SOUTH_THERM6_N renamed SOUTH_THERM6_N
- C218 pad 1: GND -> GNDS
- C219 pad 1: GND -> GNDS
- C224 pad 1: GND -> GNDS
- C225 pad 1: GND -> GNDS
- C306 pad 2: GND -> GNDS
- C313 pad 2: GND -> GNDS
- C314 pad 1: GND -> GNDS
- C315 pad 1: GND -> GNDS
- C320 pad 1: GND -> GNDS
- C321 pad 1: GND -> GNDS
- C326 pad 2: GND -> GNDS
- C327 pad 2: GND -> GNDS
- C328 pad 2: GND -> GNDS
- C329 pad 2: GND -> GNDS
- C330 pad 2: GND -> GNDS
- C331 pad 2: GND -> GNDS
- C332 pad 2: GND -> GNDS
- C333 pad 2: GND -> GNDS
- C334 pad 2: GND -> GNDS
- C335 pad 2: GND -> GNDS
- C336 pad 2: GND -> GNDS
- C337 pad 2: GND -> GNDS
- C338 pad 2: GND -> GNDS
- Q400 pad 2: Net-(Q400-Pad2) -> GND
- R110 pad 2: /MCU/STM32_RX_J -> /MCU/STM32_RX_P
- R111 pad 2: /MCU/STM32_TX_J -> /MCU/STM32_TX_N
- R201 pad 2: /South(Master)_BQ/SOUTH_CELL5 -> SOUTH_CELL_5
- R202 pad 2: /South(Master)_BQ/SOUTH_CELL4 -> SOUTH_CELL_5
- R205 pad 2: /South(Master)_BQ/SOUTH_CELL1 -> SOUTH_CELL_1
- R208 pad 2: /South(Master)_BQ/SOUTH_CELL5 -> SOUTH_CELL_5
- R209 pad 2: /South(Master)_BQ/SOUTH_CELL4 -> SOUTH_CELL_5
- R212 pad 2: /South(Master)_BQ/SOUTH_CELL1 -> SOUTH_CELL_1
- R301 pad 2: /NORTH_BQ/NORTH_CELL5 -> NORTH_CELL_5
- R302 pad 2: /NORTH_BQ/NORTH_CELL4 -> NORTH_CELL_5
- R305 pad 2: /NORTH_BQ/NORTH_CELL1 -> SOUTH_CELL_1
- R308 pad 2: /NORTH_BQ/NORTH_CELL5 -> NORTH_CELL_5
- R309 pad 2: /NORTH_BQ/NORTH_CELL4 -> NORTH_CELL_5
- R312 pad 2: /NORTH_BQ/NORTH_CELL1 -> SOUTH_CELL_1
- R329 pad 2: GND -> GNDS
- R330 pad 2: GND -> GNDS
- R331 pad 2: GND -> GNDS
- R332 pad 2: GND -> GNDS
- R333 pad 2: GND -> GNDS
- R334 pad 2: GND -> GNDS
- R335 pad 2: GND -> GNDS
- R403 pad 2: Net-(Q400-Pad2) -> GND
- U1 pad 15: GND -> GNDS
- U1 pad 26: GND -> GNDS
- U1 pad 35: GND -> GNDS
- U1 pad 43: /NORTH_BQ/NORTH_THERM1_P -> NORTH_THERM1_P
- U1 pad 45: GND -> GNDS
- U101 pad 24: /MCU/DIAGS_TX_P -> /MCU/STM32_TX_N
- U101 pad 25: /MCU/DIAGS_RX_N -> /MCU/STM32_RX_P
- U101 pad 29: Net-(U101-Pad29) -> /MCU/DIAGS_TX_P
- U101 pad 30: Net-(U101-Pad30) -> /MCU/DIAGS_RX_N
- U200 pad 43: /South(Master)_BQ/SOUTH_THERM1_P -> SOUTH_THERM1_P

Commit message: For review call
Parts:
- added C115: 11mF, Capacitor_SMD:C_1210_3225Metric, F.Cu at (342.2, 13.3)
- added D110: GN, LED_SMD:LED_0603_1608Metric, F.Cu at (321.3, 32.1)
- added D111: GN, LED_SMD:LED_0603_1608Metric, F.Cu at (325.3, 32.1)
- added D112: PMEG6002EJ, Diode_SMD:D_SOD-323F, F.Cu at (312.8, 32.2)
- added D113: D_Small, Diode_SMD:D_SOD-323F, F.Cu at (317.1, 32.2)
- added D2: PMEG6002EJ, Diode_SMD:D_SOD-323F, F.Cu at (308.6, 32.2)
- added D3: PMEG6002EJ, Diode_SMD:D_SOD-323F, F.Cu at (341.5, 16.9)
- added J104: CAN_CONN, Connector_Dsub:DSUB-9_Female_Horizontal_P2.77x2.84mm_EdgePinOffset4.94mm_Housed_MountingHolesOffset7.48mm, F.Cu at (311.4, 26.6)
- added R126: 0, Resistor_SMD:R_0603_1608Metric, F.Cu at (341.4, 19.6)
- added R127: 470, Resistor_SMD:R_0603_1608Metric, F.Cu at (329.3, 32.0)
- added R128: 470, Resistor_SMD:R_0603_1608Metric, F.Cu at (341.4, 22.1)
- D100, D104, D105, D106: value LED -> OG
- D107, D108: value LED -> RD
- moved H0 300.6 mm to (307.7, -1.70)
- moved H1 300.6 mm to (307.7, -8.65)
- moved H2 300.6 mm to (300.8, -1.70)
- moved H3 300.6 mm to (300.8, -8.65)
- moved R1 300.6 mm to (317.2, -7.58)
- moved R2 300.6 mm to (313.2, -2.56)
- moved R3 300.6 mm to (313.2, -0.05)
- moved R4 300.6 mm to (317.2, -5.07)
- moved R5 300.6 mm to (321.2, -7.58)
- moved R6 300.6 mm to (313.2, -7.58)
- moved R7 300.6 mm to (317.2, -2.56)
- moved R8 300.6 mm to (317.2, -0.05)
- moved TP3 275.9 mm to (300.5, 37.0)
- moved C313 156.8 mm to (36.5, 156.8)
- moved C312 151.7 mm to (36.7, 150.7)
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- renumbered C115 to C116, D2 to D109, J3 to J102
Connections:
- net /INPUT_OUTPUT/BATT_FAULT renamed BATT_FAULT
- net /INPUT_OUTPUT/CHG_FAULT renamed CHG_FAULT
- net /INPUT_OUTPUT/DIS_FAULT renamed DIS_FAULT
- C219 pad 2: /South(Master)_BQ/NORTH_COML_N -> NORTH_COML_N
- C225 pad 2: /South(Master)_BQ/NORTH_FAULTL_N -> NORTH_FAULTL_N
- C317 pad 2: /NORTH_BQ/SOUTH_COMN_N -> SOUTH_COMN_N
- C323 pad 2: /NORTH_BQ/SOUTH_FAULTN_N -> SOUTH_FAULTN_N
- C400 pad 1: /INPUT_OUTPUT/I_CHG -> I_CHG
- C402 pad 1: /INPUT_OUTPUT/V_CHG -> V_CHG
- C403 pad 1: /INPUT_OUTPUT/I_DIS -> I_DIS
- C404 pad 1: /INPUT_OUTPUT/V_DIS -> V_DIS
- C406 pad 1: /INPUT_OUTPUT/I_BATT -> I_BATT
- C407 pad 1: /INPUT_OUTPUT/V_BATT -> V_BATT
- J100 pad 1: +3V3 -> Net-(D2-Pad1)
- J102 pad 1: +3V3 -> Net-(D112-Pad2)
- Q400 pad 1: /INPUT_OUTPUT/CHG_ON -> CHG_ON
- Q401 pad 1: /INPUT_OUTPUT/DIS_ON -> DIS_ON
- Q402 pad 1: /INPUT_OUTPUT/BATT_ON -> BATT_ON
- R101 pad 2: /MCU/A1 -> I_DIS
- R102 pad 2: /MCU/A2 -> V_DIS
- R103 pad 2: /MCU/A3 -> I_CHG
- R104 pad 2: /MCU/A4 -> V_BATT
- R105 pad 2: /MCU/A5 -> I_BATT
- R106 pad 2: /MCU/A6 -> V_CHG
- R107 pad 2: /MCU/A7 -> DIS_ON
- R108 pad 2: /MCU/A9 -> CHG_ON
- R109 pad 2: /MCU/A11 -> BATT_ON
- R110 pad 1: /MCU/STM32_RX -> STM32_RX
- R111 pad 1: /MCU/STM32_TX -> STM32_TX
- R112 pad 1: /MCU/~BMS_FAULT -> ~BMS_FAULT
- R113 pad 1: /MCU/BMS_WAKEUP -> BMS_WAKEUP
- R215 pad 1: /South(Master)_BQ/NORTH_COML_P -> NORTH_COML_P
- R217 pad 1: /South(Master)_BQ/NORTH_COML_N -> NORTH_COML_N
- R219 pad 1: /South(Master)_BQ/NORTH_COML_N -> NORTH_COML_N
- R219 pad 2: /South(Master)_BQ/NORTH_COML_P -> NORTH_COML_P
- R223 pad 1: /South(Master)_BQ/NORTH_FAULTL_P -> NORTH_FAULTL_P
- R224 pad 1: /South(Master)_BQ/NORTH_FAULTL_N -> NORTH_FAULTL_N
- R225 pad 1: /South(Master)_BQ/NORTH_FAULTL_N -> NORTH_FAULTL_N
- R225 pad 2: /South(Master)_BQ/NORTH_FAULTL_P -> NORTH_FAULTL_P
- R234 pad 2: /South(Master)_BQ/STM32_RX -> STM32_RX
- R235 pad 2: /South(Master)_BQ/STM32_TX -> STM32_TX
- R236 pad 2: /South(Master)_BQ/~BMS_FAULT -> ~BMS_FAULT
- R237 pad 2: /South(Master)_BQ/BMS_WAKEUP -> BMS_WAKEUP
- R317 pad 1: /NORTH_BQ/SOUTH_COMN_P -> SOUTH_COMN_P
- R318 pad 1: /NORTH_BQ/SOUTH_COMN_N -> SOUTH_COMN_N
- R319 pad 1: /NORTH_BQ/SOUTH_COMN_N -> SOUTH_COMN_N
- R319 pad 2: /NORTH_BQ/SOUTH_COMN_P -> SOUTH_COMN_P
- R321 pad 1: /NORTH_BQ/SOUTH_FAULTN_P -> SOUTH_FAULTN_P
- R324 pad 1: /NORTH_BQ/SOUTH_FAULTN_N -> SOUTH_FAULTN_N
- R325 pad 1: /NORTH_BQ/SOUTH_FAULTN_N -> SOUTH_FAULTN_N
- R325 pad 2: /NORTH_BQ/SOUTH_FAULTN_P -> SOUTH_FAULTN_P
- R401 pad 1: /INPUT_OUTPUT/V_CHG -> V_CHG
- R402 pad 2: /INPUT_OUTPUT/V_CHG -> V_CHG
- R403 pad 1: /INPUT_OUTPUT/CHG_ON -> CHG_ON
- R409 pad 1: /INPUT_OUTPUT/V_DIS -> V_DIS
- R410 pad 2: /INPUT_OUTPUT/V_DIS -> V_DIS
- R412 pad 1: /INPUT_OUTPUT/V_BATT -> V_BATT
- R414 pad 2: /INPUT_OUTPUT/V_BATT -> V_BATT
- R415 pad 1: /INPUT_OUTPUT/BATT_ON -> BATT_ON
- R418 pad 1: /INPUT_OUTPUT/DIS_ON -> DIS_ON
- TP1 pad 1: /MCU/BMS_WAKEUP -> BMS_WAKEUP
- TP106 pad 1: /MCU/STM32_RX -> STM32_RX
- TP107 pad 1: /MCU/STM32_TX -> STM32_TX
- TP108 pad 1: /MCU/~BMS_FAULT -> ~BMS_FAULT
- TP201 pad 1: /South(Master)_BQ/NORTH_COML_P -> NORTH_COML_P
- TP203 pad 1: /South(Master)_BQ/NORTH_COML_N -> NORTH_COML_N
- TP205 pad 1: /South(Master)_BQ/NORTH_FAULTL_P -> NORTH_FAULTL_P
- TP207 pad 1: /South(Master)_BQ/NORTH_FAULTL_N -> NORTH_FAULTL_N
- TP301 pad 1: /NORTH_BQ/SOUTH_COMN_P -> SOUTH_COMN_P
- TP303 pad 1: /NORTH_BQ/SOUTH_COMN_N -> SOUTH_COMN_N
- TP306 pad 1: /NORTH_BQ/SOUTH_FAULTN_P -> SOUTH_FAULTN_P
- TP307 pad 1: /NORTH_BQ/SOUTH_FAULTN_N -> SOUTH_FAULTN_N
- U1 pad 17: /NORTH_BQ/NORTH_COML_N -> NORTH_COML_N
- U1 pad 18: /NORTH_BQ/NORTH_COML_P -> NORTH_COML_P
- U1 pad 19: /NORTH_BQ/NORTH_FAULTL_P -> NORTH_FAULTL_P
- U1 pad 20: /NORTH_BQ/NORTH_FAULTL_N -> NORTH_FAULTL_N
- U101 pad 1: +3V3 -> Net-(C115-Pad1)
- U200 pad 16: /South(Master)_BQ/BMS_WAKEUP -> BMS_WAKEUP
- U200 pad 17: /South(Master)_BQ/SOUTH_COMN_N -> SOUTH_COMN_N
- U200 pad 18: /South(Master)_BQ/SOUTH_COMN_P -> SOUTH_COMN_P
- U200 pad 19: /South(Master)_BQ/SOUTH_FAULTN_P -> SOUTH_FAULTN_P
- U200 pad 20: /South(Master)_BQ/SOUTH_FAULTN_N -> SOUTH_FAULTN_N
- U200 pad 40: /South(Master)_BQ/STM32_RX -> STM32_RX
- U200 pad 41: /South(Master)_BQ/STM32_TX -> STM32_TX
- U200 pad 42: /South(Master)_BQ/~BMS_FAULT -> ~BMS_FAULT

Commit message: prelim layout ???
Parts:
- R328, R329: moved to B.Cu
- moved U402 302.5 mm to (41.1, 119.8), turned to 90 degrees
- moved F402 301.6 mm to (36.6, 120.8)
- moved D1 293.0 mm to (41.8, 126.6), turned to 180 degrees
- moved J402 279.2 mm to (20.5, 128.8)
- moved U403 277.5 mm to (48.3, 122.5), turned to 270 degrees
- moved C101 274.3 mm to (76.6, 103.8), turned to 90 degrees
- moved U100 268.0 mm to (79.5, 103.5)
- moved C100 266.0 mm to (78.3, 100.2), turned to 90 degrees
- moved TP3 265.1 mm to (35.5, 43.0)
- moved U404 261.0 mm to (80.9, 125.2), turned to 180 degrees
- moved U400 259.8 mm to (90.4, 108.4), turned to 90 degrees
- moved F100 259.6 mm to (76.8, 100.2), turned to 90 degrees
- moved F400 255.3 mm to (95.0, 108.9), turned to 180 degrees
- moved U405 254.1 mm to (89.7, 124.4), turned to 90 degrees
- moved R128 254.0 mm to (88.3, 43.9), turned to 90 degrees
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Connections:
- J500 pad 1: SOUTH_CELL_6 -> Net-(J500-Pad1)
- J500 pad 10: SOUTH_THERM1_P -> Net-(J500-Pad10)
- J500 pad 11: SOUTH_THERM2_N -> Net-(J500-Pad11)
- J500 pad 12: SOUTH_THERM1_P -> SOUTH_CELL_0
- J500 pad 13: SOUTH_THERM3_N -> SOUTH_CELL_1
- J500 pad 14: SOUTH_THERM1_P -> SOUTH_CELL_2
- J500 pad 15: SOUTH_THERM4_N -> SOUTH_CELL_3
- J500 pad 16: SOUTH_THERM1_P -> SOUTH_CELL_4
- J500 pad 17: SOUTH_THERM5_N -> SOUTH_CELL_5
- J500 pad 18: SOUTH_THERM1_P -> SOUTH_CELL_6
- J500 pad 19: SOUTH_THERM6_N -> Net-(J500-Pad19)
- J500 pad 2: SOUTH_CELL_5 -> Net-(J500-Pad2)
- J500 pad 3: SOUTH_CELL_5 -> Net-(J500-Pad3)
- J500 pad 4: SOUTH_CELL_3 -> Net-(J500-Pad4)
- J500 pad 5: SOUTH_CELL_2 -> Net-(J500-Pad5)
- J500 pad 6: SOUTH_CELL_1 -> Net-(J500-Pad6)
- J500 pad 7: SOUTH_CELL_0 -> Net-(J500-Pad7)
- J500 pad 8: SOUTH_THERM1_P -> Net-(J500-Pad8)
- J500 pad 9: SOUTH_THERM1_N -> Net-(J500-Pad9)
- R202 pad 2: SOUTH_CELL_5 -> SOUTH_CELL_4
- R209 pad 2: SOUTH_CELL_5 -> SOUTH_CELL_4
Routing:
- net Net-(C226-Pad1): track 0.00 -> 11.9 mm
- net /South(Master)_BQ/SOUTH_BAL_CELL5_FILT: track 0.00 -> 5.71 mm
- net /South(Master)_BQ/SOUTH_BAL_CELL2_FILT: track 0.00 -> 5.65 mm
- net /South(Master)_BQ/SOUTH_BAL_CELL4_FILT: track 0.00 -> 5.64 mm
- net /South(Master)_BQ/SOUTH_BAL_CELL0_FILT: track 0.00 -> 5.62 mm
- net /South(Master)_BQ/SOUTH_BAL_CELL1_FILT: track 0.00 -> 5.60 mm
- net /South(Master)_BQ/SOUTH_BAL_CELL3_FILT: track 0.00 -> 5.34 mm
- net /South(Master)_BQ/SOUTH_BAT: track 0.00 -> 4.20 mm
- net Net-(C231-Pad1): track 0.00 -> 3.88 mm
- net /South(Master)_BQ/SOUTH_TAP_CELL5_FILT: track 0.00 -> 3.50 mm
- net /South(Master)_BQ/SOUTH_BAL_CELL6_FILT: track 0.00 -> 3.02 mm
- net /South(Master)_BQ/SOUTH_LDOIN: track 0.00 -> 2.99 mm
- net /South(Master)_BQ/SOUTH_TAP_CELL3_FILT: track 0.00 -> 2.97 mm
- net /South(Master)_BQ/SOUTH_TAP_CELL2_FILT: track 0.00 -> 2.97 mm
- net /South(Master)_BQ/SOUTH_TAP_CELL1_FILT: track 0.00 -> 2.97 mm
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Other:
- copper layers 2 -> 4

Commit message: (maybe) final placement V1,0
Parts:
- removed the J102 at (206.6, 57.1)
- removed TP1: BMS_WAKEUP, TestPoint:TestPoint_Bridge_Pitch2.54mm_Drill1.0mm
- removed TP200: SOUTH_COMH_P, TestPoint:TestPoint_Bridge_Pitch2.54mm_Drill1.0mm
- removed TP201: NORTH_COML_P, TestPoint:TestPoint_Bridge_Pitch2.54mm_Drill1.0mm
- removed TP202: SOUTH_COMH_N, TestPoint:TestPoint_Bridge_Pitch2.54mm_Drill1.0mm
- removed TP203: NORTH_COML_N, TestPoint:TestPoint_Bridge_Pitch2.54mm_Drill1.0mm
- removed TP204: SOUTH_FAULTH_P, TestPoint:TestPoint_Bridge_Pitch2.54mm_Drill1.0mm
- removed TP205: NORTH_FAULTL_P, TestPoint:TestPoint_Bridge_Pitch2.54mm_Drill1.0mm
- removed TP206: SOUTH_FAULTH_N, TestPoint:TestPoint_Bridge_Pitch2.54mm_Drill1.0mm
- removed TP207: NORTH_FAULTL_N, TestPoint:TestPoint_Bridge_Pitch2.54mm_Drill1.0mm
- removed TP300: NORTH_COMH_P, TestPoint:TestPoint_Bridge_Pitch2.54mm_Drill1.0mm
- removed TP301: SOUTH_COML_P, TestPoint:TestPoint_Bridge_Pitch2.54mm_Drill1.0mm
- removed TP302: NORTH_COMH_N, TestPoint:TestPoint_Bridge_Pitch2.54mm_Drill1.0mm
- removed TP303: SOUTH_COMN_N, TestPoint:TestPoint_Bridge_Pitch2.54mm_Drill1.0mm
- removed TP304: NORTH_FAULTH_P, TestPoint:TestPoint_Bridge_Pitch2.54mm_Drill1.0mm
- removed TP305: NORTH_FAULTH_N, TestPoint:TestPoint_Bridge_Pitch2.54mm_Drill1.0mm
- removed TP306: SOUTH_FAULTN_P, TestPoint:TestPoint_Bridge_Pitch2.54mm_Drill1.0mm
- removed TP307: SOUTH_FAULTN_N, TestPoint:TestPoint_Bridge_Pitch2.54mm_Drill1.0mm
- added TP109: BMS_WAKEUP, TestPoint:TestPoint_Pad_D1.0mm, F.Cu at (56.9, 39.1)
- added TP401: POWER_MIX, TestPoint:TestPoint_Pad_D1.0mm, F.Cu at (67.4, 129.7)
- added TP402: DISCHARGE, TestPoint:TestPoint_Pad_D1.0mm, F.Cu at (92.6, 122.7)
- TP100, TP102, TP103, TP106, TP107, TP108, TP110, TP111: footprint TestPoint:TestPoint_Bridge_Pitch2.54mm_Drill1.0mm -> TestPoint:TestPoint_Pad_D1.0mm
- TP101: value 3V3 RAIL -> 3V3_RAIL; footprint TestPoint:TestPoint_Bridge_Pitch2.54mm_Drill1.0mm -> TestPoint:TestPoint_Pad_D1.0mm
- U400, U402, U405: footprint Sensor_Current:Allegro_QFN-12-10-1EP_3x3mm_P0.5mm -> Milpitas_BMS:Allegro_QFN-12-10-1EP_3x3mm_P0.5mm
- moved R7 206.6 mm to (25.3, 133.8)
- moved R8 206.0 mm to (25.4, 135.4)
- moved H3 202.2 mm to (20.3, 134.6)
- moved R104 195.1 mm to (38.6, 129.2), turned to 90 degrees
- moved R109 171.6 mm to (50.5, 118.2), turned to 90 degrees
- moved R1 167.1 mm to (26.0, 38.4)
- moved R105 166.3 mm to (36.1, 116.7), turned to 270 degrees
- moved H0 162.0 mm to (20.3, 37.7)
- moved R2 161.8 mm to (26.0, 36.8)
- moved R5 160.5 mm to (102.7, 135.5), turned to 180 degrees
- moved R111 156.5 mm to (61.0, 43.3)
- moved R6 154.8 mm to (102.7, 134.0), turned to 180 degrees
- moved R110 151.7 mm to (61.0, 45.3)
- moved R121 151.4 mm to (70.3, 68.8), turned to 90 degrees
- moved TP108 149.3 mm to (56.9, 41.2)
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- renumbered D2 to D114
Connections:
- net /MCU/DIAGS_RX_N renamed /MCU/DIAGS_N
- net /MCU/STM32_RX_P renamed /MCU/STM32_UART_J_P
- net /MCU/STM32_TX_N renamed /MCU/STM32_UART_J_N
- net /MCU/XTAL32_OUT_N renamed /MCU/XTAL32_IN_N
- net /MCU/XTAL_IN_P renamed /MCU/XTAL_P
- net /MCU/XTAL_OUT_N renamed /MCU/XTAL_N
- net Net-(C214-Pad1) renamed /South(Master)_BQ/S_COMH_LS_P
- net Net-(C215-Pad1) renamed /South(Master)_BQ/S_COMH_LS_N
- net Net-(C221-Pad1) renamed /South(Master)_BQ/S_FAULTH_LS_P
- net Net-(C223-Pad1) renamed /South(Master)_BQ/S_FAULTH_LS_N
- net Net-(C315-Pad2) renamed /NORTH_BQ/N_COMH_LS_P
- net Net-(C319-Pad2) renamed /NORTH_BQ/N_COMH_LS_N
- net Net-(C321-Pad2) renamed /NORTH_BQ/N_FAULTH_LS_P
- net Net-(C324-Pad2) renamed /NORTH_BQ/N_FAULTH_LS_N
- net STM32_RX renamed STM32_UART_P
- net STM32_TX renamed STM32_UART_N
- C303 pad 2: Net-(C303-Pad2) -> /NORTH_BQ/NORTH_TAP_CELL2_FILT
- C304 pad 1: Net-(C303-Pad2) -> /NORTH_BQ/NORTH_TAP_CELL2_FILT
- J102 pad 1: Net-(D112-Pad2) -> /MCU/DIAGS_P
- J102 pad 2: /MCU/DIAGS_TX_P -> Net-(D112-Pad2)
- J104 pad 2: /MCU/CAN_H_P -> /MCU/CAN_P
- J104 pad 3: /MCU/CAN_L_N -> /MCU/CAN_N
- J104 pad 4: /MCU/CAN_SH -> /MCU/CAN_P
- J104 pad 5: /MCU/CAN_H_P -> /MCU/CAN_SH
- J104 pad 6: /MCU/CAN_L_N -> Net-(J104-Pad6)
- J104 pad 8: Net-(J104-Pad8) -> /MCU/CAN_N
- JP100 pad 1: /MCU/CAN_H_P -> /MCU/CAN_P
- R115 pad 1: /MCU/CAN_L_N -> /MCU/CAN_N
- R125 pad 1: /MCU/DIAGS_TX_P -> /MCU/DIAGS_P
- R226 pad 2: +BATT -> SOUTH_CELL_6
- R227 pad 2: +BATT -> SOUTH_CELL_6
- R304 pad 1: Net-(C303-Pad2) -> /NORTH_BQ/NORTH_TAP_CELL2_FILT
- TP104 pad 1: /MCU/CAN_H_P -> /MCU/CAN_P
- TP105 pad 1: /MCU/CAN_L_N -> /MCU/CAN_N
- U101 pad 29: /MCU/DIAGS_TX_P -> /MCU/DIAGS_P
- U102 pad 6: /MCU/CAN_L_N -> /MCU/CAN_N
- U102 pad 7: /MCU/CAN_H_P -> /MCU/CAN_P
Routing:
- net STM32_UART_P: track 0.00 -> 10.3 mm
- net STM32_UART_N: track 0.00 -> 10.1 mm
- net /MCU/XTAL_P: track 0.00 -> 5.00 mm
- net Net-(R417-Pad1): track 0.00 -> 4.95 mm
- net Net-(R10-Pad2): track 0.00 -> 4.28 mm
- net Net-(R9-Pad2): track 0.00 -> 4.20 mm
- net +3V3: track 0.00 -> 3.53 mm
- net /South(Master)_BQ/SOUTH_FAULTH_N: track 0.00 -> 3.06 mm
- net /South(Master)_BQ/SOUTH_COMH_N: track 0.00 -> 3.03 mm
- net Net-(C221-Pad2): track 0.00 -> 2.94 mm
- net Net-(Q402-Pad3): track 0.00 -> 2.16 mm
- net Net-(R416-Pad1): track 0.00 -> 2.13 mm
- net CHG_ON: track 0.00 -> 1.57 mm
- net /MCU/CAN_TX_P: track 0.00 -> 1.53 mm
- net Net-(D110-Pad2): track 0.00 -> 1.52 mm
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Other:
- board outline added: 94 x 103.4 mm
- board text added: "BATT."
- board text added: "CHG."
- board text added: "DIS."
- board text added: "STATE MACHINE: LEFT | RIGHT 00: STANDBY 01: DISCHARGE 10: CHARGE 11: FAULT"
