File: Milpitas_BMS/PCB/Cell_Tap_Pinout.sch (KiCad schematic (older format))
At the start: 16 parts, among them J1 Conn_01x02, J2 Conn_01x20, J500 SOUTH CELL CONN, J501 NORTH CELL CONN

Commit message: Ordered board. Hopefully it's all gucci prada
Other:
- note added: "Wiring Diagram"
- note removed: "PINOUT TBD UNTIL LAYOUT BEGINS"
- note removed: "WIRING DIAGRAM BY CELL BLOCK"
- moved on the sheet: J500, J501
