File: Milpitas_BMS/PCB/INPUT_OUTPUT.sch (KiCad schematic (older format))
At the start: 46 parts, among them J400 CHG INPUT, J401 POWER_OUTPUT, J402 BATT_PWR_INPUT, Q400 RU1J002YNTCL, Q401 RU1J002YNTCL, Q402 RU1J002YNTCL, U400 ACS711, U401 BTS6163DAUMA1, U402 ACS711, U403 BTS6163DAUMA1, U404 BTS6163DAUMA1, U405 ACS711

Commit message: Ordered board. Hopefully it's all gucci prada
Parts:
- added BATT1: BATT_RAIL, TestPoint:TestPoint_Pad_D1.0mm, symbol Connector:TestPoint
- added C440: 0.47uF, Capacitor_SMD:C_0603_1608Metric, symbol Device:C_Small
- C400, C401, C402, C403, C404, C405, C406, C407, C408: Digikey (none) -> 1292-1451-1-ND
- R400, R402, R403, R405, R407, R408, R410, R411, R414, R415, R417, R418: Digikey (none) -> 311-1.0KGRCT-ND
- R401, R409, R412: Digikey (none) -> RMCF0603FT140KCT-ND
- R404, R406, R416: Digikey (none) -> A129685CT-ND
- renumbered TP400 to CHARGER1, TP402 to DISCHARGE1, TP401 to MIXED1
Connections:
- net +BATT: now also BATT1.1
- net DIS_ON: now also C440.1
- net GND: now also C440.2
Other:
- moved on the sheet: CHARGER1, DISCHARGE1, MIXED1
Changed lines of the file:
@@
 F 2 "Resistor_SMD:R_0603_1608Metric" V 4480 4750 50  0001 C CNN
 F 3 "~" H 4550 4750 50  0001 C CNN
+F 4 "311-1.0KGRCT-ND" H 4550 4750 50  0001 C CNN "Digikey"
 	1    4550 4750
 	1    0    0    -1
@@
 F 2 "Resistor_SMD:R_0603_1608Metric" V 4280 2500 50  0001 C CNN
 F 3 "~" H 4350 2500 50  0001 C CNN
+F 4 "311-1.0KGRCT-ND" H 4350 2500 50  0001 C CNN "Digikey"
 	1    4350 2500
 	1    0    0    -1
@@
 F 2 "Resistor_SMD:R_0603_1608Metric" V 6930 2500 50  0001 C CNN
 F 3 "~" H 7000 2500 50  0001 C CNN
+F 4 "311-1.0KGRCT-ND" H 7000 2500 50  0001 C CNN "Digikey"
 	1    7000 2500
 	1    0    0    -1
@@
 F 2 "Resistor_SMD:R_0603_1608Metric" V 6730 2250 50  0001 C CNN
 F 3 "~" H 6800 2250 50  0001 C CNN
+F 4 "A129685CT-ND" H 6800 2250 50  0001 C CNN "Digikey"
 	1    6800 2250
 	1    0    0    -1
@@
 F 2 "Resistor_SMD:R_0603_1608Metric" V 6330 2800 50  0001 C CNN
 F 3 "~" H 6400 2800 50  0001 C CNN
+F 4 "311-1.0KGRCT-ND" H 6400 2800 50  0001 C CNN "Digikey"
 	1    6400 2800
 	1    0    0    -1
@@
 	6400 2600 6500 2600
 Wire Wire Line
-	6400 2600 6050 2600
+	6400 2600 6250 2600
 Connection ~ 6400 2600
 Text Label 6050 2600 0    39   ~ 0
@@
 F 2 "Resistor_SMD:R_0603_1608Metric" V 4230 4500 50  0001 C CNN
 F 3 "~" H 4300 4500 50  0001 C CNN
+F 4 "A129685CT-ND" H 4300 4500 50  0001 C CNN "Digikey"
 	1    4300 4500
 	1    0    0    -1
@@
 F 2 "Resistor_SMD:R_0603_1608Metric" V 3830 5050 50  0001 C CNN
 F 3 "~" H 3900 5050 50  0001 C CNN
+F 4 "311-1.0KGRCT-ND" H 3900 5050 50  0001 C CNN "Digikey"
 	1    3900 5050
 	1    0    0    -1
@@
 F 3 "~" H 2700 1450 50  0001 C CNN
 F 4 "10V" H 2700 1450 50  0001 C CNN "Voltage"
+F 5 "1292-1451-1-ND" H 2700 1450 50  0001 C CNN "Digikey"
 	1    2700 1450
 	1    0    0    -1
@@
 F 2 "Resistor_SMD:R_0603_1608Metric" V 1580 1650 50  0001 C CNN
 F 3 "~" H 1650 1650 50  0001 C CNN
+F 4 "311-1.0KGRCT-ND" H 1650 1650 50  0001 C CNN "Digikey"
 	1    1650 1650
 	1    0    0    -1
@@
 F 3 "~" H 1650 2250 50  0001 C CNN
 F 4 "10V" H 1650 2250 50  0001 C CNN "Voltage"
+F 5 "1292-1451-1-ND" H 1650 2250 50  0001 C CNN "Digikey"
 	1    1650 2250
 	1    0    0    -1
@@
 F 3 "~" H 2750 3700 50  0001 C CNN
 F 4 "10V" H 2750 3700 50  0001 C CNN "Voltage"
+F 5 "1292-1451-1-ND" H 2750 3700 50  0001 C CNN "Digikey"
 	1    2750 3700
 	1    0    0    -1
@@
 F 2 "Resistor_SMD:R_0603_1608Metric" V 1630 3900 50  0001 C CNN
 F 3 "~" H 1700 3900 50  0001 C CNN
+F 4 "311-1.0KGRCT-ND" H 1700 3900 50  0001 C CNN "Digikey"
 	1    1700 3900
 	1    0    0    -1
@@
 F 3 "~" H 1700 4500 50  0001 C CNN
 F 4 "10V" H 1700 4500 50  0001 C CNN "Voltage"
+F 5 "1292-1451-1-ND" H 1700 4500 50  0001 C CNN "Digikey"
 	1    1700 4500
 	1    0    0    -1
@@
 Wire Wire Line
 	1700 4050 1700 4250
-Wire Wire Line
-	1900 4100 1450 4100
 Text Label 1350 4350 0    39   ~ 0
 I_BATT
@@
 F 2 "Resistor_SMD:R_0603_1608Metric" V 4030 2200 50  0001 C CNN
 F 3 "~" H 4100 2200 50  0001 C CNN
+F 4 "A129685CT-ND" H 4100 2200 50  0001 C CNN "Digikey"
 	1    4100 2200
 	1    0    0    -1
@@
 F 2 "Resistor_SMD:R_0603_1608Metric" V 3630 2750 50  0001 C CNN
 F 3 "~" H 3700 2750 50  0001 C CNN
+F 4 "311-1.0KGRCT-ND" H 3700 2750 50  0001 C CNN "Digikey"
 	1    3700 2750
 	1    0    0    -1
@@
 F 2 "Resistor_SMD:R_0603_1608Metric" V 3180 2600 50  0001 C CNN
 F 3 "~" H 3250 2600 50  0001 C CNN
+F 4 "311-1.0KGRCT-ND" H 3250 2600 50  0001 C CNN "Digikey"
 	1    3250 2600
 	1    0    0    1
@@
 F 2 "Resistor_SMD:R_0603_1608Metric" V 3180 2150 50  0001 C CNN
 F 3 "~" H 3250 2150 50  0001 C CNN
+F 4 "RMCF0603FT140KCT-ND" H 3250 2150 50  0001 C CNN "Digikey"
 	1    3250 2150
 	1    0    0    1
@@
 F 3 "~" H 8450 2250 50  0001 C CNN
 F 4 "10V" H 8450 2250 50  0001 C CNN "Voltage"
+F 5 "1292-1451-1-ND" H 8450 2250 50  0001 C CNN "Digikey"
 	1    8450 2250
 	1    0    0    -1
@@
 F 2 "Resistor_SMD:R_0603_1608Metric" V 8380 1650 50  0001 C CNN
 F 3 "~" H 8450 1650 50  0001 C CNN
+F 4 "311-1.0KGRCT-ND" H 8450 1650 50  0001 C CNN "Digikey"
 	1    8450 1650
 	1    0    0    -1
@@
 F 3 "~" H 9500 1450 50  0001 C CNN
 F 4 "10V" H 9500 1450 50  0001 C CNN "Voltage"
+F 5 "1292-1451-1-ND" H 9500 1450 50  0001 C CNN "Digikey"
 	1    9500 1450
 	1    0    0    -1
@@
 F 2 "Resistor_SMD:R_0603_1608Metric" V 10130 2700 50  0001 C CNN
 F 3 "~" H 10200 2700 50  0001 C CNN
+F 4 "311-1.0KGRCT-ND" H 10200 2700 50  0001 C CNN "Digikey"
 	1    10200 2700
 	1    0    0    1
@@
 F 2 "Resistor_SMD:R_0603_1608Metric" V 10130 2300 50  0001 C CNN
 F 3 "~" H 10200 2300 50  0001 C CNN
+F 4 "RMCF0603FT140KCT-ND" H 10200 2300 50  0001 C CNN "Digikey"
 	1    10200 2300
 	1    0    0    1
@@
 F 3 "~" H 9800 2700 50  0001 C CNN
 F 4 "10V" H 9800 2700 50  0001 C CNN "Voltage"
+F 5 "1292-1451-1-ND" H 9800 2700 50  0001 C CNN "Digikey"
 	1    9800 2700
 	1    0    0    -1
@@
 F 2 "Resistor_SMD:R_0603_1608Metric" V 3330 4950 50  0001 C CNN
 F 3 "~" H 3400 4950 50  0001 C CNN
+F 4 "311-1.0KGRCT-ND" H 3400 4950 50  0001 C CNN "Digikey"
 	1    3400 4950
 	1    0    0    1
@@
 F 2 "Resistor_SMD:R_0603_1608Metric" V 3330 4550 50  0001 C CNN
 F 3 "~" H 3400 4550 50  0001 C CNN
+F 4 "RMCF0603FT140KCT-ND" H 3400 4550 50  0001 C CNN "Digikey"
 	1    3400 4550
 	1    0    0    1
@@
 F 3 "~" H 3000 4950 50  0001 C CNN
 F 4 "10V" H 3000 4950 50  0001 C CNN "Voltage"
+F 5 "1292-1451-1-ND" H 3000 4950 50  0001 C CNN "Digikey"
 	1    3000 4950
 	1    0    0    -1
@@
 F 3 "~" H 2850 2600 50  0001 C CNN
 F 4 "10V" H 2850 2600 50  0001 C CNN "Voltage"
+F 5 "1292-1451-1-ND" H 2850 2600 50  0001 C CNN "Digikey"
 	1    2850 2600
 	1    0    0    -1
@@
 Connection ~ 3400 4100
 Wire Wire Line
-	3400 4100 4050 4100
+	3400 4100 3650 4100
 Wire Wire Line
 	6800 2100 6800 2050
@@
 XT30
 $Comp
-L Connector:TestPoint TP400
+L Connector:TestPoint CHARGER1
 U 1 1 6262E257
-P 1350 1250
-F 0 "TP400" H 1408 1368 50  0000 L CNN
-F 1 "CHARGER" H 1408 1277 50  0000 L CNN
-F 2 "TestPoint:TestPoint_Pad_D1.0mm" H 1550 1250 50  0001 C CNN
-F 3 "~" H 1550 1250 50  0001 C CNN
-	1    1350 1250
-	1    0    0    -1
-$EndComp
-Wire Wire Line
-	1350 1850 1350 1250
+P 1350 1550
+F 0 "CHARGER1" H 1408 1668 50  0000 L CNN
+F 1 "CHARGER" H 1408 1577 50  0001 L CNN
+F 2 "TestPoint:TestPoint_Pad_D1.0mm" H 1550 1550 50  0001 C CNN
+F 3 "~" H 1550 1550 50  0001 C CNN
+	1    1350 1550
+	1    0    0    -1
+$EndComp
+Wire Wire Line
+	1350 1850 1350 1550
 Connection ~ 1350 1850
 Wire Wire Line
 	1350 1850 1850 1850
 Wire Wire Line
-	10200 1850 10200 1250
-Wire Wire Line
-	5900 1850 5900 1300
+	10200 1850 10200 1650
+Wire Wire Line
+	5900 1850 5900 1750
 Text Label 6100 1850 0    39   ~ 0
 MIXED_PWR_PLANE
@@
 L Connector:TestPoint TP?
 U 1 1 5FCA12D8
-P 5900 1300
+P 5900 1750
 AR Path="/5FD707DF/5FCA12D8" Ref="TP?"  Part="1"
-AR Path="/5FD4A06E/5FCA12D8" Ref="TP401"  Part="1"
-F 0 "TP401" H 5958 1418 50  0000 L CNN
-F 1 "POWER_MIX" H 5958 1327 50  0000 L CNN
-F 2 "TestPoint:TestPoint_Pad_D1.0mm" H 6100 1300 50  0001 C CNN
-F 3 "" H 6100 1300 50  0001 C CNN
-F 4 "" H 5900 1300 50  0001 C CNN "Digikey"
-	1    5900 1300
+AR Path="/5FD4A06E/5FCA12D8" Ref="MIXED1"  Part="1"
+F 0 "MIXED1" H 5958 1868 50  0000 L CNN
+F 1 "POWER_MIX" H 5958 1777 50  0001 L CNN
+F 2 "TestPoint:TestPoint_Pad_D1.0mm" H 6100 1750 50  0001 C CNN
+F 3 "" H 6100 1750 50  0001 C CNN
+F 4 "" H 5900 1750 50  0001 C CNN "Digikey"
+	1    5900 1750
 	1    0    0    -1
 $EndComp
@@
 L Connector:TestPoint TP?
 U 1 1 5FCA7AF1
-P 10200 1250
+P 10200 1650
 AR Path="/5FD707DF/5FCA7AF1" Ref="TP?"  Part="1"
-AR Path="/5FD4A06E/5FCA7AF1" Ref="TP402"  Part="1"
-F 0 "TP402" H 10258 1368 50  0000 L CNN
-F 1 "DISCHARGE" H 10258 1277 50  0000 L CNN
-F 2 "TestPoint:TestPoint_Pad_D1.0mm" H 10400 1250 50  0001 C CNN
-F 3 "" H 10400 1250 50  0001 C CNN
-F 4 "" H 10200 1250 50  0001 C CNN "Digikey"
-	1    10200 1250
-	1    0    0    -1
-$EndComp
+AR Path="/5FD4A06E/5FCA7AF1" Ref="DISCHARGE1"  Part="1"
+F 0 "DISCHARGE1" H 10258 1768 50  0000 L CNN
+F 1 "DISCHARGE" H 10258 1677 50  0001 L CNN
+F 2 "TestPoint:TestPoint_Pad_D1.0mm" H 10400 1650 50  0001 C CNN
+F 3 "" H 10400 1650 50  0001 C CNN
+F 4 "" H 10200 1650 50  0001 C CNN "Digikey"
+	1    10200 1650
+	1    0    0    -1
+$EndComp
+$Comp
+L Connector:TestPoint TP?
+U 1 1 5EA610C1
+P 3650 3950
+AR Path="/5FD707DF/5EA610C1" Ref="TP?"  Part="1"
+AR Path="/5FD4A06E/5EA610C1" Ref="BATT1"  Part="1"
+F 0 "BATT1" H 3708 4068 50  0000 L CNN
+F 1 "BATT_RAIL" H 3708 3977 50  0000 L CNN
+F 2 "TestPoint:TestPoint_Pad_D1.0mm" H 3850 3950 50  0001 C CNN
+F 3 "" H 3850 3950 50  0001 C CNN
+F 4 "" H 3650 3950 50  0001 C CNN "Digikey"
+	1    3650 3950
+	1    0    0    -1
+$EndComp
+Wire Wire Line
+	3650 3950 3650 4100
+Wire Wire Line
+	1450 4100 1900 4100
+Connection ~ 3650 4100
+Wire Wire Line
+	3650 4100 4050 4100
+$Comp
+L Device:C_Small C440
+U 1 1 5EB9AB16
+P 6250 2800
+F 0 "C440" H 5950 2850 50  0000 L CNN
+F 1 "0.47uF" H 5950 2750 50  0000 L CNN
+F 2 "Capacitor_SMD:C_0603_1608Metric" H 6250 2800 50  0001 C CNN
+F 3 "~" H 6250 2800 50  0001 C CNN
+F 4 "10V" H 6250 2800 50  0001 C CNN "Voltage"
+F 5 "1292-1451-1-ND" H 6250 2800 50  0001 C CNN "Digikey"
+	1    6250 2800
+	1    0    0    -1
+$EndComp
+Wire Wire Line
+	6250 2700 6250 2600
+Connection ~ 6250 2600
+Wire Wire Line
+	6250 2600 6050 2600
+Wire Wire Line
+	6250 2900 6250 3000
+Wire Wire Line
+	6250 3000 6400 3000
+Connection ~ 6400 3000
 $EndSCHEMATC
