File: Milpitas_BMS/PCB/MCU.sch (KiCad schematic (older format))
At the start: 89 parts, among them J100 JTAG, J102 DIAGS_CON, J104 CAN_CONN, SW100 SW_SPST, SW101 SW_SPST, U100 MIC5283-3.3ML-TR, U101 STM32F303RETx, U102 SN65HVD232, Y1 32.768kHz, Y2 16MHz

Commit message: Ordered board. Hopefully it's all gucci prada
Parts:
- removed TP100: BATT_RAIL, TestPoint:TestPoint_Pad_D1.0mm, symbol Connector:TestPoint
- C100, C102: Digikey (none) -> 1276-1860-1-ND
- C101: Digikey (none) -> 399-7845-1-ND
- C103, C104, C105, C106, C107, C108, C109, C116: Digikey (none) -> 1292-1451-1-ND
- C110: Digikey (none) -> 399-7880-1-ND
- C111, C112: Digikey (none) -> 490-11478-1-ND
- C113, C114: Digikey (none) -> 490-9670-1-ND
- R10, R101, R102, R103, R104, R105, R106, R107, R108, R109, R110, R111, R112, R113, R114, R126, R9: Digikey (none) -> 311-0.0GRCT-ND
- R100, R116, R117, R118: Digikey (none) -> A129673CT-ND
- R115: Digikey (none) -> 311-120HRCT-ND
- R119, R120: Digikey (none) -> 311-30GRCT-ND
- R121, R122, R123, R124, R125: Digikey (none) -> 311-10KGRCT-ND
- R127, R128: Digikey (none) -> 311-470GRCT-ND
- renumbered TP101 to 3V3_RAIL1, TP106 to STM32_RX1, TP107 to STM32_RX2, TP109 to WAKEUP1, TP108 to ~FAULT1
Other:
- note added: "CAN Pinout"
- note added: "DIAGS_N = STM32_TX\nDIAGS_P = STM32_RX\n"
- note removed: "Following GPIO Subject to Layout preference. \n(Associated filtering/pullups/downs are on local page)\n(Only MCU protection circuitry shown) \n- CHG_ON\n- GHG_FAULT\n- DIS_ON\n- DIS_FAULT\n- BATT_ON\n- BATT_FAULT\n- BMS_FAULT\n- BMS_WAKEUP\n- CHG_LED\n- DIS_LED\n- BATT_LED\n- SM0\n- SM1\n- USR_BUTTON"
- moved on the sheet: STM32_RX1, STM32_RX2, ~{FAULT1}
