File: Milpitas_BMS/PCB/Milpitas_BMS.kicad_pcb (KiCad board)
At the start: 4 copper layers, 89.8 x 103.5 mm, 325 parts, among them J100 JTAG, J102 DIAGS_CON, J104 CAN_CONN, J500 SOUTH CELL CONN, J501 NORTH CELL CONN, Q400 RU1J002YNTCL, Q401 RU1J002YNTCL, Q402 RU1J002YNTCL, SW100 SW_SPST, SW101 SW_SPST, U1 BQ79606, U100 MIC5283-3.3ML-TR, U101 STM32F303RETx, U102 SN65HVD232, U200 BQ79606, U400 ACS711, U401 BTS6163DAUMA1, U402 ACS711, U403 BTS6163DAUMA1, U404 BTS6163DAUMA1, U405 ACS711, Y1 32.768kHz, Y2 16MHz

Commit message: Ordered board. Hopefully it's all gucci prada
Parts:
- removed the G*** at (127.3, 144.7)
- removed the G*** at (125.3, 144.4)
- 3V3_RAIL: renamed from 3V3 RAIL
- TP110: renamed from 32.768 kHz
- TP111: renamed from 16 MHz
- TP2: renamed from ISOLATED GROUND
- TP3: renamed from REGULAR GROUND
- moved BATT 0.14 mm to (141.4, 147.3)
- renumbered TERM to JP100, STM32_TX to STM32_RX, CAN_TX to TP102, CAN_RX to TP103, WAKEUP to WAKEUP1, ~FAULT to ~FAULT1
Connections:
- U1 pad 49: (no net) -> GNDS
- U100 pad 9: (no net) -> GND
- U200 pad 49: (no net) -> GND
Routing:
- net GND: track 184.3 -> 200.9 mm, vias 100 -> 101
- net +BATT: track 66.7 -> 68.2 mm, vias 8 -> 5
- net Net-(F402-Pad1): vias 4 -> 0
- net /INPUT_OUTPUT/BATT_RAW: vias 3 -> 0
Other:
- rule pad_to_mask_clearance: 0.051 -> 0
- rule solder_mask_min_width: 0.25 -> 0.005
- board text added: "DIAGS: MCU TX | 3V3 MCU RX | GND"
