File: Milpitas_BMS/PCB/NORTH_BQS.sch (KiCad schematic (older format))
At the start: 83 parts, among them U1 BQ79606

Commit message: Ordered board. Hopefully it's all gucci prada
Parts:
- C300, C301, C302, C303, C304, C305, C306, C307, C308, C309, C310, C311, C312, C313, C333, C334, C335, C336, C337, C338: Digikey (none) -> 1292-1451-1-ND
- C314, C315, C316, C317, C320, C321, C322, C323: Digikey (none) -> 1276-2310-1-ND
- C318, C319, C324, C325: Digikey (none) -> 399-7880-1-ND
- C326, C327: Digikey (none) -> 445-7462-1-ND
- C328, C329, C330, C331, C332: Digikey (none) -> 1276-1085-1-ND
- R300, R301, R302, R303, R304, R305, R306: Digikey (none) -> 541-3318-1-ND
- R307, R308, R309, R310, R311, R312, R313: value 12 -> 25; Digikey (none) -> 541-2654-1-ND
- R314, R319, R323, R325: Digikey (none) -> 311-10KGRCT-ND
- R315, R316, R317, R318, R320, R321, R322, R324: Digikey (none) -> 2019-RN73H1JTTD49R3B25CT-ND
- R326: Digikey (none) -> 541-2655-1-ND
- R327: Digikey (none) -> 311-100HRCT-ND
- R328, R329: Digikey (none) -> 311-0.0GRCT-ND
- R330, R331, R332, R333, R334, R335: Digikey (none) -> RMCF0603FT13K7CT-ND
- R336, R337, R338, R339, R340, R341: Digikey (none) -> 311-1.0KGRCT-ND
Connections:
- net GNDS: now also U1.49 (PAD)
