File: Milpitas_BMS/PCB/South(Master)_BQ.sch (KiCad schematic (older format))
At the start: 86 parts, among them U200 BQ79606

Commit message: Ordered board. Hopefully it's all gucci prada
Parts:
- C200, C201, C202, C203, C204, C205, C206, C207, C208, C209, C210, C211, C212, C213, C234, C235, C236, C237, C238, C239: Digikey (none) -> 1292-1451-1-ND
- C214, C215, C221, C223: Digikey (none) -> 399-7880-1-ND
- C216, C217, C218, C219, C220, C222, C224, C225: Digikey (none) -> 1276-2310-1-ND
- C226, C227, C228, C229, C230, C231: Digikey (none) -> 1276-1085-1-ND
- C232, C233: Digikey (none) -> 445-7462-1-ND
- R200, R201, R202, R203, R204, R205, R206: Digikey (none) -> 541-3318-1-ND
- R207, R208, R209, R210, R211, R212, R213: value 12 -> 25; Digikey (none) -> 541-2654-1-ND
- R214, R215, R216, R217, R221, R222, R223, R224: Digikey (none) -> 2019-RN73H1JTTD49R3B25CT-ND
- R218, R219, R220, R225, R234, R235, R236, R237: Digikey (none) -> 311-10KGRCT-ND
- R226: Digikey (none) -> 541-2655-1-ND
- R227: Digikey (none) -> 311-100HRCT-ND
- R228, R229, R230, R231, R232, R233: Digikey (none) -> RMCF0603FT13K7CT-ND
- R238, R239, R240, R250, R251, R252: Digikey (none) -> 311-1.0KGRCT-ND
Connections:
- net GND: now also U200.49 (PAD)
